Commit message: Fixed robot moving

File: franka_ros/panda_moveit_config/config/panda_arm_hand.srdf.xacro (robot description, xacro)
@@ -27,4 +27,5 @@
     <joint name="panda_joint6" value="1.571" />
     <joint name="panda_joint7" value="0.785" />
+    <!-- <joint name="panda_finger_joint1" value="0" /> -->
   </group_state>
   <!--END EFFECTOR: Purpose: Represent information about an end effector.-->
